File: pcbs/lara_hat_v2/lara_hat_v2.kicad_pcb (KiCad board)
At the start: 2 copper layers, 85 x 56 mm, 29 parts, among them J1 Raspberry_Pi_4, J2 Conn_RoboClaw, J3 Conn_Dynamixel, J4 Conn_01x02_Pin, J5 12V in, J6 LED_JST, J7 I2C_JST, U1 MCP2515-xSO, U2 SN65HVD230, U3 74LVC2G241, U5 12V-5V-Buck, Y1 8MHz

Commit message: hat update
Parts:
- C4: footprint Capacitor_SMD:C_Elec_4x5.4 -> Capacitor_SMD:C_0805_2012Metric_Pad1.18x1.45mm_HandSolder
- moved C4 1.26 mm to (140.4, 114.8)
Routing:
- net +3V3: track 114.4 -> 149.2 mm, vias 4 -> 5
- net GND: track 28.1 -> 0.00 mm
Other:
- outline, holes or cut-outs redrawn
- board text added: "12V"
- board text added: "GND"
- board text removed: "12V IN"

Commit message: hat update
Parts:
- U3: footprint Package_SO:VSSOP-8_3x3mm_P0.65mm -> Package_SO:VSSOP-8_2.3x2mm_P0.5mm
- moved J2 1.69 mm to (137.1, 122.5)
- moved U3 0.32 mm to (148.3, 114.5)
Routing:
- net GND: track 0.00 -> 2.44 mm, vias 3 -> 8
- net Net-(J1-GPIO14/UART_TXD): track 72.8 -> 70.9 mm, vias 0 -> 1
- net Net-(J1-GPIO15/UART_RXD): track 66.6 -> 66.0 mm
- net Net-(J1-ID_SD_I2C0/GPIO00): track 44.1 -> 44.7 mm
- net +3V3: track 149.2 -> 149.8 mm
- net Net-(J1-SCL_I2C1/GPIO03): track 71.5 -> 71.0 mm
Other:
- board text added: "G"
- board text added: "Rx"
- board text added: "Tx"

Commit message: pcb update
Parts:
- added R6: 4.7k, Resistor_SMD:R_0805_2012Metric_Pad1.20x1.40mm_HandSolder, F.Cu at (169.8, 118.8)
- added R7: 4.7k, Resistor_SMD:R_0805_2012Metric_Pad1.20x1.40mm_HandSolder, F.Cu at (169.8, 115.3)
- J5: value 12V in -> 1723104202; footprint TerminalBlock:TerminalBlock_MaiXu_MX126-5.0-02P_1x02_P5.00mm -> Molex_Ultra-Fit_Horizontal:CONN_1723102000_02_MOL
- moved J5 23.0 mm to (191.3, 112.3)
- moved J7 21.2 mm to (175.6, 124.2)
- moved U5 3.23 mm to (187.5, 95.8)
Routing:
- net +12V: track 50.9 -> 73.6 mm
- net +3V3: track 149.8 -> 136.9 mm
- net Net-(J1-GPIO12/PWM0): track 60.5 -> 51.7 mm
- net Net-(J1-GPIO13/PWM1): track 61.5 -> 52.8 mm
- net +5V: track 73.1 -> 74.5 mm
- net GND: vias 8 -> 9
