File: pcbs/lara_hat_v2/lara_hat_v2.kicad_sch (KiCad schematic)
At the start: 27 parts, among them J1 Raspberry_Pi_4, J2 Conn_RoboClaw, J3 Conn_Dynamixel, J4 Conn_01x02_Pin, J5 12V in, J6 LED_JST, J7 I2C_JST, U1 MCP2515-xSO, U2 SN65HVD230, U3 74LVC2G241, U5 12V-5V-Buck, Y1 8MHz

Commit message: hat update
Parts:
- C4: footprint Capacitor_SMD:C_Elec_4x5.4 -> Capacitor_SMD:C_0805_2012Metric_Pad1.18x1.45mm_HandSolder
Changed lines of the file:
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@@
 			)
 		)
-		(property "Footprint" "Capacitor_SMD:C_Elec_4x5.4"
+		(property "Footprint" "Capacitor_SMD:C_0805_2012Metric_Pad1.18x1.45mm_HandSolder"
 			(at 247.3452 43.18 0)
 			(effects

Commit message: hat update
Parts:
- U3: footprint Package_SO:VSSOP-8_3x3mm_P0.65mm -> Package_SO:VSSOP-8_2.3x2mm_P0.5mm
Changed lines of the file:
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@@
 			)
 		)
-		(property "Footprint" "Package_SO:VSSOP-8_3x3mm_P0.65mm"
+		(property "Footprint" "Package_SO:VSSOP-8_2.3x2mm_P0.5mm"
 			(at 212.09 39.37 0)
 			(effects
@@
 		(on_board yes)
 		(dnp no)
-		(fields_autoplaced yes)
 		(property "Reference" "U3"
 			(at 171.45 102.87 0)
@@
 			)
 		)
-		(property "Footprint" "Package_SO:VSSOP-8_3x3mm_P0.65mm"
-			(at 172.72 93.98 0)
-			(effects
-				(font
-					(size 1.27 1.27)
-				)
-				(hide yes)
+		(property "Footprint" "Package_SO:VSSOP-8_2.3x2mm_P0.5mm"
+			(at 197.612 99.568 0)
+			(effects
+				(font
+					(size 1.27 1.27)
+				)
 			)
 		)
@@
 			)
 		)
-		(property "Footprint" "Package_SO:VSSOP-8_3x3mm_P0.65mm"
+		(property "Footprint" "Package_SO:VSSOP-8_2.3x2mm_P0.5mm"
 			(at 172.72 58.42 0)
 			(effects

Commit message: pcb update
Parts:
- added R6, R7: 4.7k, Resistor_SMD:R_0805_2012Metric_Pad1.20x1.40mm_HandSolder, symbol Device:R
Connections:
- net +3V3: now also R6.2, R7.2
- net at J1.32 (GPIO12/PWM0), J7.3 (Pin_3): now also R6.1
- net at J1.33 (GPIO13/PWM1), J7.4 (Pin_4): now also R7.1

Commit message: pcb update
Parts:
- removed J5: 12V in, TerminalBlock:TerminalBlock_MaiXu_MX126-5.0-02P_1x02_P5.00mm, symbol Connector:Screw_Terminal_01x02
- added J5: 1723104202, CONN_1723102000_02_MOL, symbol Molex_Ultra-Fit_Horizontal:1723104202
Connections:
- net +12V: now also J5.1
- net GND: now also J5.2
Changed lines of the file:
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@@
 	(wire
 		(pts
-			(xy 101.6 35.56) (xy 96.52 35.56)
+			(xy 96.52 35.56) (xy 104.14 35.56)
 		)
 		(stroke
@@
 	(wire
 		(pts
-			(xy 96.52 33.02) (xy 101.6 33.02)
+			(xy 96.52 33.02) (xy 104.14 33.02)
 		)
 		(stroke
@@
 	)
 	(symbol
-		(lib_id "Connector:Screw_Terminal_01x02")
-		(at 106.68 33.02 0)
-		(unit 1)
-		(exclude_from_sim no)
-		(in_bom yes)
-		(on_board yes)
-		(dnp no)
-		(fields_autoplaced yes)
-		(property "Reference" "J5"
-			(at 109.22 33.0199 0)
-			(effects
-				(font
-					(size 1.27 1.27)
-				)
-				(justify left)
-			)
-		)
-		(property "Value" "12V in"
-			(at 109.22 35.5599 0)
-			(effects
-				(font
-					(size 1.27 1.27)
-				)
-				(justify left)
-			)
-		)
-		(property "Footprint" "TerminalBlock:TerminalBlock_MaiXu_MX126-5.0-02P_1x02_P5.00mm"
-			(at 106.68 33.02 0)
-			(effects
-				(font
-					(size 1.27 1.27)
-				)
-				(hide yes)
-			)
-		)
-		(property "Datasheet" "~"
-			(at 106.68 33.02 0)
-			(effects
-				(font
-					(size 1.27 1.27)
-				)
-				(hide yes)
-			)
-		)
-		(property "Description" "Generic screw terminal, single row, 01x02, script generated (kicad-library-utils/schlib/autogen/connector/)"
-			(at 106.68 33.02 0)
-			(effects
-				(font
-					(size 1.27 1.27)
-				)
-				(hide yes)
-			)
-		)
-		(pin "1"
-		)
-		(pin "2"
-		)
-		(instances
-			(project ""
-				(path "/439a50f9-54cc-4d05-be8a-2234828ed849"
-					(reference "J5")
-					(unit 1)
-				)
-			)
-		)
-	)
-	(symbol
 		(lib_id "Device:LED")
 		(at 31.75 96.52 90)
@@
 					(unit 1)
 				)
+			)
+		)
+	)
+	(symbol
+		(lib_id "Molex_Ultra-Fit_Horizontal:1723104202")
+		(at 104.14 33.02 0)
+		(unit 1)
+		(exclude_from_sim no)
+		(in_bom yes)
+		(on_board yes)
+		(dnp no)
+		(property "Reference" "J5"
+			(at 118.11 33.0199 0)
+			(effects
+				(font
+					(size 1.524 1.524)
+				)
+				(justify left)
+			)
+		)
+		(property "Value" "1723104202"
+			(at 105.664 28.702 0)
+			(effects
+				(font
+					(size 1.524 1.524)
+				)
+				(justify left)
+			)
+		)
+		(property "Footprint" "CONN_1723102000_02_MOL"
+			(at 104.14 33.02 0)
+			(effects
+				(font
+					(size 1.27 1.27)
+					(italic yes)
+				)
+				(hide yes)
+			)
+		)
+		(property "Datasheet" "https://www.molex.com/en-us/products/part-detail-pdf/1723104202?display=pdf"
+			(at 104.14 33.02 0)
+			(effects
+				(font
+					(size 1.27 1.27)
+					(italic yes)
+				)
+				(hide yes)
+			)
+		)
+		(property "Description" ""
+			(at 104.14 33.02 0)
+			(effects
+				(font
+					(size 1.27 1.27)
+				)
+				(hide yes)
+			)
+		)
+		(pin "2"
+		)
+		(pin "1"
+		)
+		(instances
+			(project ""
+				(path "/439a50f9-54cc-4d05-be8a-2234828ed849"
+					(reference "J5")
+					(unit 1)
+				)

Commit message: updates
Other:
- company: (none) -> ETSIDI UPM
- title: (none) -> LARA HAT
Changed lines of the file:
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@@
 	(generator_version "9.0")
 	(paper "A4")
+	(title_block
+		(title "LARA HAT")
+		(rev "V2")
+		(company "ETSIDI UPM")
+	)
 	(junction
 		(at 190.5 58.42)
@@
 		)
 		(instances
-			(project ""
+			(project "lara_hat_v2"
 				(path "/439a50f9-54cc-4d05-be8a-2234828ed849"
 					(reference "U3")
@@
 		)
 		(instances
-			(project ""
+			(project "lara_hat_v2"
 				(path "/439a50f9-54cc-4d05-be8a-2234828ed849"
 					(reference "J4")
@@
 		)
 		(instances
-			(project ""
+			(project "lara_hat_v2"
 				(path "/439a50f9-54cc-4d05-be8a-2234828ed849"
 					(reference "R2")
@@
 		)
 		(instances
-			(project ""
+			(project "lara_hat_v2"
 				(path "/439a50f9-54cc-4d05-be8a-2234828ed849"
 					(reference "#PWR021")
@@
 		)
 		(instances
-			(project ""
+			(project "lara_hat_v2"
 				(path "/439a50f9-54cc-4d05-be8a-2234828ed849"
 					(reference "C3")
@@
 		)
 		(instances
-			(project "LARA_hat"
+			(project "lara_hat_v2"
 				(path "/439a50f9-54cc-4d05-be8a-2234828ed849"
 					(reference "C4")
@@
 		)
 		(instances
-			(project ""
+			(project "lara_hat_v2"
 				(path "/439a50f9-54cc-4d05-be8a-2234828ed849"
 					(reference "#PWR017")
@@
 		)
 		(instances
-			(project "LARA_hat"
+			(project "lara_hat_v2"
 				(path "/439a50f9-54cc-4d05-be8a-2234828ed849"
 					(reference "#PWR026")
@@
 		)
 		(instances
-			(project ""
+			(project "lara_hat_v2"
 				(path "/439a50f9-54cc-4d05-be8a-2234828ed849"
 					(reference "#PWR08")
@@
 		)
 		(instances
-			(project ""
+			(project "lara_hat_v2"
 				(path "/439a50f9-54cc-4d05-be8a-2234828ed849"
 					(reference "U3")
@@
 		)
 		(instances
-			(project ""
+			(project "lara_hat_v2"
 				(path "/439a50f9-54cc-4d05-be8a-2234828ed849"
 					(reference "Y1")
@@
 		)
 		(instances
-			(project ""
+			(project "lara_hat_v2"
 				(path "/439a50f9-54cc-4d05-be8a-2234828ed849"
 					(reference "#PWR06")
@@
 		)
 		(instances
-			(project ""
+			(project "lara_hat_v2"
 				(path "/439a50f9-54cc-4d05-be8a-2234828ed849"
 					(reference "C1")
@@
 		)
 		(instances
-			(project ""
+			(project "lara_hat_v2"
 				(path "/439a50f9-54cc-4d05-be8a-2234828ed849"
 					(reference "#PWR020")
@@
 		)
 		(instances
-			(project "LARA_hat"
+			(project "lara_hat_v2"
 				(path "/439a50f9-54cc-4d05-be8a-2234828ed849"
 					(reference "J6")
@@
 		)
 		(instances
-			(project ""
+			(project "lara_hat_v2"
 				(path "/439a50f9-54cc-4d05-be8a-2234828ed849"
 					(reference "#PWR07")
@@
 		)
 		(instances
-			(project ""
+			(project "lara_hat_v2"
 				(path "/439a50f9-54cc-4d05-be8a-2234828ed849"
 					(reference "#PWR012")
@@
 		)
 		(instances
-			(project ""
+			(project "lara_hat_v2"
 				(path "/439a50f9-54cc-4d05-be8a-2234828ed849"
 					(reference "J3")
@@
 		)
 		(instances
-			(project "LARA_hat"
+			(project "lara_hat_v2"
 				(path "/439a50f9-54cc-4d05-be8a-2234828ed849"
 					(reference "D4")
@@
 		)
 		(instances
-			(project ""
+			(project "lara_hat_v2"
 				(path "/439a50f9-54cc-4d05-be8a-2234828ed849"
 					(reference "U2")
@@
 		)
 		(instances
-			(project "LARA_hat"
+			(project "lara_hat_v2"
 				(path "/439a50f9-54cc-4d05-be8a-2234828ed849"
 					(reference "R5")
@@
 		)
 		(instances
-			(project ""
+			(project "lara_hat_v2"
 				(path "/439a50f9-54cc-4d05-be8a-2234828ed849"
 					(reference "U3")
@@
 		)
 		(instances
-			(project "LARA_hat"
+			(project "lara_hat_v2"
 				(path "/439a50f9-54cc-4d05-be8a-2234828ed849"
 					(reference "R8")
@@
 		)
 		(instances
-			(project ""
+			(project "lara_hat_v2"
 				(path "/439a50f9-54cc-4d05-be8a-2234828ed849"
 					(reference "#PWR04")
@@
 		)
 		(instances
-			(project "LARA_hat"
+			(project "lara_hat_v2"
 				(path "/439a50f9-54cc-4d05-be8a-2234828ed849"
 					(reference "D3")
@@
 		)
 		(instances
-			(project ""
+			(project "lara_hat_v2"
 				(path "/439a50f9-54cc-4d05-be8a-2234828ed849"
 					(reference "J2")
@@
 		)
 		(instances
-			(project ""
+			(project "lara_hat_v2"
 				(path "/439a50f9-54cc-4d05-be8a-2234828ed849"
 					(reference "#PWR03")
@@
 		)
 		(instances
-			(project ""
+			(project "lara_hat_v2"
 				(path "/439a50f9-54cc-4d05-be8a-2234828ed849"
 					(reference "R3")
@@
 		)
 		(instances
-			(project ""
+			(project "lara_hat_v2"
 				(path "/439a50f9-54cc-4d05-be8a-2234828ed849"
 					(reference "#PWR02")
@@
 		)
 		(instances
-			(project ""
+			(project "lara_hat_v2"
 				(path "/439a50f9-54cc-4d05-be8a-2234828ed849"
 					(reference "#PWR05")
@@
 		)
 		(instances
-			(project ""
+			(project "lara_hat_v2"
 				(path "/439a50f9-54cc-4d05-be8a-2234828ed849"
 					(reference "J5")
@@
 		)
 		(instances
-			(project ""
+			(project "lara_hat_v2"
 				(path "/439a50f9-54cc-4d05-be8a-2234828ed849"
 					(reference "C2")
@@
 		)
 		(instances
-			(project "LARA_hat"
+			(project "lara_hat_v2"
 				(path "/439a50f9-54cc-4d05-be8a-2234828ed849"
 					(reference "D5")
@@
 		)
 		(instances
-			(project ""
+			(project "lara_hat_v2"
 				(path "/439a50f9-54cc-4d05-be8a-2234828ed849"
 					(reference "#PWR011")
@@
 		)
 		(instances
-			(project "LARA_hat"
+			(project "lara_hat_v2"
 				(path "/439a50f9-54cc-4d05-be8a-2234828ed849"
 					(reference "#PWR024")
@@
 		)
 		(instances
-			(project ""
+			(project "lara_hat_v2"
 				(path "/439a50f9-54cc-4d05-be8a-2234828ed849"
 					(reference "J7")
@@
 		)
 		(instances
-			(project ""
+			(project "lara_hat_v2"
 				(path "/439a50f9-54cc-4d05-be8a-2234828ed849"
 					(reference "#PWR016")
@@
 		)
 		(instances
-			(project ""
+			(project "lara_hat_v2"
 				(path "/439a50f9-54cc-4d05-be8a-2234828ed849"
 					(reference "#PWR019")
@@
 		)
 		(instances
-			(project ""
+			(project "lara_hat_v2"
 				(path "/439a50f9-54cc-4d05-be8a-2234828ed849"
 					(reference "#PWR09")
@@
 		)
 		(instances
-			(project ""
+			(project "lara_hat_v2"
 				(path "/439a50f9-54cc-4d05-be8a-2234828ed849"
 					(reference "R1")
@@
 		)
 		(instances
-			(project ""
+			(project "lara_hat_v2"
 				(path "/439a50f9-54cc-4d05-be8a-2234828ed849"
 					(reference "#PWR014")
@@
 		)
 		(instances
-			(project ""
+			(project "lara_hat_v2"
 				(path "/439a50f9-54cc-4d05-be8a-2234828ed849"
 					(reference "#PWR027")
@@
 		)
 		(instances
-			(project ""
+			(project "lara_hat_v2"
 				(path "/439a50f9-54cc-4d05-be8a-2234828ed849"
 					(reference "J1")
@@
 		)
 		(instances
-			(project "LARA_hat"
+			(project "lara_hat_v2"
 				(path "/439a50f9-54cc-4d05-be8a-2234828ed849"
 					(reference "R9")
@@
 		)
 		(instances
-			(project "LARA_hat"
+			(project "lara_hat_v2"
 				(path "/439a50f9-54cc-4d05-be8a-2234828ed849"
 					(reference "#PWR025")
@@
 		)
 		(instances
-			(project ""
+			(project "lara_hat_v2"
 				(path "/439a50f9-54cc-4d05-be8a-2234828ed849"
 					(reference "U1")
@@
 		)
 		(instances
-			(project ""
+			(project "lara_hat_v2"
 				(path "/439a50f9-54cc-4d05-be8a-2234828ed849"
 					(reference "#PWR01")
@@
 		)
 		(instances
-			(project "LARA_hat"
+			(project "lara_hat_v2"
 				(path "/439a50f9-54cc-4d05-be8a-2234828ed849"
 					(reference "R10")
@@
 		)
 		(instances
-			(project ""
+			(project "lara_hat_v2"
 				(path "/439a50f9-54cc-4d05-be8a-2234828ed849"
 					(reference "#PWR010")
@@
 		)
 		(instances
-			(project ""
+			(project "lara_hat_v2"
 				(path "/439a50f9-54cc-4d05-be8a-2234828ed849"
 					(reference "R4")
@@
 		)
 		(instances
-			(project ""
+			(project "lara_hat_v2"
 				(path "/439a50f9-54cc-4d05-be8a-2234828ed849"
 					(reference "U5")
@@
 		)
 		(instances
-			(project ""
+			(project "lara_hat_v2"
 				(path "/439a50f9-54cc-4d05-be8a-2234828ed849"
 					(reference "#PWR015")
@@
 		)
 		(instances
-			(project ""
+			(project "lara_hat_v2"
 				(path "/439a50f9-54cc-4d05-be8a-2234828ed849"
 					(reference "#PWR018")
